Commit message: renamed files for consistency and fixed paths in urdf files

File: gki_sensors_description/urdf/sick_rfu620.urdf.xacro (robot description, xacro)
@@ -32,11 +32,10 @@
             <texture filename="package://gki_sensors_description/meshes/sick_rfu620_diffuse_map.png"/>
           </material>
+        </visual>
         <collision>
-        </visual>
           <origin xyz="0 0 -0.021" rpy="0 0 0" />
           <geometry>
-          <box size="0.05 0.05 0.07" />
-          <!--<mesh filename="package://gki_sensors_description/meshes/hokuyo_urg.stl"/>-->
-        </geometry>
+            <box size="0.05 0.05 0.07" />
+          </geometry>
         </collision>
       </link>

Commit message: bug fixes in sick_rfu620

File: gki_sensors_description/urdf/sick_rfu620.urdf.xacro (robot description, xacro)
@@ -29,6 +29,7 @@
             <mesh filename="package://gki_sensors_description/meshes/sick_rfu620.dae"/>
           </geometry>
-          <material name="${name}_material">
-            <texture filename="package://gki_sensors_description/meshes/sick_rfu620_diffuse_map.png"/>
+          <material name="${name}_texture">
+            <color rgb="255 0 0" alpha="1.0"/>
+            <!--<texture filename="package://gki_sensors_description/meshes/sick_rfu620_diffuse_map.png"/>-->
           </material>
         </visual>
@@ -36,5 +37,5 @@
           <origin xyz="0 0 -0.021" rpy="0 0 0" />
           <geometry>
-            <box size="0.05 0.05 0.07" />
+            <box size="0.13 0.13 0.07" />
           </geometry>
         </collision>
