Commit message: improved axis215 model, added logitech c525 urdf

File: gki_sensors_description/urdf/axis215.urdf.xacro (robot description, xacro)
@@ -5,5 +5,5 @@
   xmlns:xacro="http://ros.org/wiki/xacro"
   >
-    <include filename="$(find turtlebot_description)/urdf/common_properties.urdf.xacro" />
+    <xacro:include filename="$(find turtlebot_description)/urdf/common_properties.urdf.xacro" />
     <xacro:macro name="axis215" params="name parent *origin">
       <joint name="${name}_joint" type="fixed">
@@ -21,5 +21,5 @@
           <origin xyz="0 0 0.0" rpy="0 0 0" />
           <geometry>
-            <mesh filename="package://gki_sensors_description/meshes/axis215.stl"/>
+            <mesh filename="package://gki_sensors_description/meshes/axis215.dae"/>
           </geometry>
           <xacro:insert_block name="material_white" />
@@ -48,5 +48,5 @@
           <limit lower="0.0" upper="1.57079632679489661922" effort="1.0" velocity="3.14" />
       </joint>
-      <!-- If optical frame is somewhat turned, put this here -->
+      <!-- If optical frame is somewhat rotated, put this here -->
       <joint name="${name}_tilt_to_optical" type="fixed">
           <origin xyz="0.0 0.0 0.0" rpy="${-M_PI/2} 0 ${-M_PI/2}" />
@@ -54,7 +54,4 @@
           <child link="${name}_optical_link"/>
       </joint>
-      <!-- axis_link is base/center of camera???
-           Finally: make sure that frame is send in axis_camera pubs for imgs and everything that has a header -->
-    <!-- Also needs to be tested for offsets/rotation + direction -->
     </xacro:macro>
 </robot>

File: gki_sensors_description/urdf/hokuyo_urg.urdf.xacro (robot description, xacro)
@@ -4,6 +4,5 @@
 xmlns:controller="http://playerstage.sourceforge.net/gazebo/xmlschema/#controller"
 xmlns:interface="http://playerstage.sourceforge.net/gazebo/xmlschema/#interface"
-  xmlns:xacro="http://ros.org/wiki/xacro"
-  >
+  xmlns:xacro="http://ros.org/wiki/xacro">
     <xacro:macro name="hokuyo_urg" params="name parent *origin ros_topic update_rate ray_count min_angle max_angle">
       <joint name="${name}_base_joint" type="fixed">
@@ -33,7 +32,7 @@
           <origin xyz="0 0 -0.021" rpy="0 0 0" />
           <geometry>
-          <box size="0.05 0.05 0.07" />
-          <!--<mesh filename="package://gki_sensors_description/meshes/hokuyo_urg.stl"/>-->
-        </geometry>
+          	<box size="0.05 0.05 0.07" />
+          	<!--<mesh filename="package://gki_sensors_description/meshes/hokuyo_urg.stl"/>-->
+        	</geometry>
         </collision>
       </link>
